Commit message: Added a pouring simulator test 1;

File: python/pybullet/data/container1.urdf.xacro (robot description, xacro)
@@ -23,5 +23,5 @@
   </xacro:macro>
   <material name="container_material">
-    <color rgba="1 0.5 1 1"/>
+    <color rgba="1 0.5 1 0.7"/>
   </material>
   <link name="base_link">
@@ -32,5 +32,5 @@
     <inertial>
       <origin rpy="0 0 0" xyz="0 0 0"/>
-      <mass value="1"/>
+      <mass value="0.2"/>
       <inertia ixx="1" ixy="0" ixz="0" iyy="1" iyz="0" izz="1"/>
     </inertial>

File: python/pybullet/data/container2.urdf.xacro (robot description, xacro)
@@ -20,5 +20,5 @@
   </xacro:macro>
   <material name="container_material">
-    <color rgba="1 1 0.5 1"/>
+    <color rgba="1 1 0.5 0.7"/>
   </material>
   <link name="base_link">
@@ -29,5 +29,5 @@
     <inertial>
       <origin rpy="0 0 0" xyz="0 0 0"/>
-      <mass value="0.7"/>
+      <mass value="0.1"/>
       <inertia ixx="1" ixy="0" ixz="0" iyy="1" iyz="0" izz="1"/>
     </inertial>
